Commit message: Added colors: red body, black wheels, blue LiDAR

File: urdf/articubot_two.xacro (robot description, xacro)
@@ -16,5 +16,5 @@
         <mesh filename="file://$(find articubot_two_description)/meshes/base_link.stl" scale="0.001 0.001 0.001"/>
       </geometry>
-      <material name="silver"/>
+      <material name="red"/>
     </visual>
     <collision>
@@ -67,5 +67,5 @@
     </collision>
   </link>
-  <!-- LIDAR -->
+  <!-- LIDAR LINK -->
   <link name="lidar_joint_1">
     <inertial>
@@ -79,5 +79,5 @@
         <mesh filename="file://$(find articubot_two_description)/meshes/lidar_joint_1.stl" scale="0.001 0.001 0.001"/>
       </geometry>
-      <material name="silver"/>
+      <material name="blue"/>
     </visual>
     <collision>
@@ -88,5 +88,5 @@
     </collision>
   </link>
-  <!-- CAMERA -->
+  <!-- CAMERA LINK -->
   <link name="camera_joint_1">
     <inertial>

File: urdf/materials.xacro (robot description, xacro)
@@ -1,9 +1,15 @@
 <?xml version="1.0"?>
 <robot xmlns:xacro="http://www.ros.org/wiki/xacro">
-  <material name="silver">
-    <color rgba="0.7 0.7 0.7 1.0"/>
+  <material name="red">
+    <color rgba="0.8 0.0 0.0 1.0"/>
   </material>
   <material name="black">
     <color rgba="0.0 0.0 0.0 1.0"/>
+  </material>
+  <material name="blue">
+    <color rgba="0.0 0.0 0.8 1.0"/>
+  </material>
+  <material name="silver">
+    <color rgba="0.7 0.7 0.7 1.0"/>
   </material>
   <material name="white">

Commit message: Clean RViz config: robot model + laser scan only

File: urdf/articubot_two.xacro (robot description, xacro)
@@ -124,9 +124,8 @@
     <dynamics damping="0.01" friction="0.01"/>
   </joint>
-  <joint name="lidar_joint" type="continuous">
+  <joint name="lidar_joint" type="fixed">
     <origin xyz="-0.057768 0.002232 0.136" rpy="0 0 0"/>
     <parent link="base_link"/>
     <child link="lidar_joint_1"/>
-    <axis xyz="0.0 0.0 1.0"/>
   </joint>
   <joint name="camera_joint" type="fixed">

Commit message: Added SLAM for map generation

File: urdf/articubot_two.xacro (robot description, xacro)
@@ -125,5 +125,5 @@
   </joint>
   <joint name="lidar_joint" type="fixed">
-    <origin xyz="-0.057768 0.002232 0.136" rpy="0 0 0"/>
+    <origin xyz="-0.057768 0.002232 0.146" rpy="0 0 0"/>
     <parent link="base_link"/>
     <child link="lidar_joint_1"/>

Commit message: Added obstacle world, updated slam and gazebo launch to use custom world

File: urdf/articubot_two.xacro (robot description, xacro)
@@ -114,5 +114,5 @@
     <parent link="base_link"/>
     <child link="left_wheel_1"/>
-    <axis xyz="0.0 1.0 0.0"/>
+    <axis xyz="0.0 -1.0 0.0"/>
     <dynamics damping="0.01" friction="0.01"/>
   </joint>
@@ -121,5 +121,5 @@
     <parent link="base_link"/>
     <child link="right_wheel_1"/>
-    <axis xyz="0.0 1.0 0.0"/>
+    <axis xyz="0.0 -1.0 0.0"/>
     <dynamics damping="0.01" friction="0.01"/>
   </joint>

Commit message: Fixed the drifting after pressing 'i' in teleop

File: urdf/articubot_two.xacro (robot description, xacro)
@@ -40,7 +40,7 @@
     </visual>
     <collision>
-      <origin xyz="-0.002232 -0.102232 -0.035" rpy="0 0 0"/>
+      <origin xyz="0.0 0.0 0.0" rpy="1.5707 0.0 0.0"/>
       <geometry>
-        <mesh filename="file://$(find articubot_two_description)/meshes/left_wheel_1.stl" scale="0.001 0.001 0.001"/>
+        <cylinder radius="0.035" length="0.025"/>
       </geometry>
     </collision>
@@ -61,7 +61,7 @@
     </visual>
     <collision>
-      <origin xyz="-0.002232 0.097768 -0.035" rpy="0 0 0"/>
+      <origin xyz="0.0 0.0 0.0" rpy="1.5707 0.0 0.0"/>
       <geometry>
-        <mesh filename="file://$(find articubot_two_description)/meshes/right_wheel_1.stl" scale="0.001 0.001 0.001"/>
+        <cylinder radius="0.035" length="0.025"/>
       </geometry>
     </collision>

Commit message: Slam totally fixed, no fluctuating

File: urdf/articubot_two.xacro (robot description, xacro)
@@ -109,4 +109,25 @@
     </collision>
   </link>
+  <!-- IMU LINK -->
+  <link name="imu_link">
+    <inertial>
+      <origin xyz="0.0 0.0 0.0" rpy="0 0 0"/>
+      <mass value="0.01"/>
+      <inertia ixx="1e-06" iyy="1e-06" izz="1e-06" ixy="0.0" iyz="0.0" ixz="0.0"/>
+    </inertial>
+    <visual>
+      <origin xyz="0 0 0" rpy="0 0 0"/>
+      <geometry>
+        <box size="0.02 0.02 0.02"/>
+      </geometry>
+      <material name="white"/>
+    </visual>
+    <collision>
+      <origin xyz="0 0 0" rpy="0 0 0"/>
+      <geometry>
+        <box size="0.02 0.02 0.02"/>
+      </geometry>
+    </collision>
+  </link>
   <!-- JOINTS -->
   <joint name="left_wheel_joint" type="continuous">
@@ -114,5 +135,5 @@
     <parent link="base_link"/>
     <child link="left_wheel_1"/>
-    <axis xyz="0.0 -1.0 0.0"/>
+    <axis xyz="0.0 1.0 0.0"/>
     <dynamics damping="0.01" friction="0.01"/>
   </joint>
@@ -121,5 +142,5 @@
     <parent link="base_link"/>
     <child link="right_wheel_1"/>
-    <axis xyz="0.0 -1.0 0.0"/>
+    <axis xyz="0.0 1.0 0.0"/>
     <dynamics damping="0.01" friction="0.01"/>
   </joint>
@@ -133,4 +154,9 @@
     <parent link="base_link"/>
     <child link="camera_joint_1"/>
+  </joint>
+  <joint name="imu_joint" type="fixed">
+    <origin xyz="0.0 0.0 0.05" rpy="0 0 0"/>
+    <parent link="base_link"/>
+    <child link="imu_link"/>
   </joint>
   <!-- ROS2 CONTROL -->
